File: Hardware/ESP32_LoRa_1_Channel_Gateway.brd (EAGLE design)
At the start: 25.4 x 45.7 mm, 84 parts, among them J3 USB, J4 QWIIC, J6 U.FL, Q1 MBT3904DW1T1, U1 3.3V, U2 CH340C, U3 ESP-WROOM-32NARROW, U4 RFM96W

Commit message: Made changes from REDS review pt 1
Parts:
- added JP1: JUMPER-SMT_2_NO_SILK, SparkFun-Jumpers:SMT-JUMPER_2_NO_SILK
- moved U$20 25.0 mm to (25.2, 6.41), flipped to the bottom
- moved FD3 23.4 mm to (24.4, 13.2), flipped to the bottom
- moved FD4 23.4 mm to (24.4, 13.2), flipped to the top
- moved U$9 23.0 mm to (25.9, 16.9), flipped to the bottom, turned to 0 degrees
- moved FD1 22.9 mm to (1.27, 44.5), flipped to the bottom
- moved FD2 22.9 mm to (1.27, 44.5), flipped to the top
- moved J1 22.9 mm to (1.27, 15.2), flipped to the bottom
- moved J2 22.9 mm to (24.1, 20.3), flipped to the bottom
- moved U$46 22.9 mm to (1.27, 10.2), flipped to the top
- moved J5 22.6 mm to (24.0, 15.2), flipped to the bottom
- moved U$45 22.6 mm to (1.40, 8.76), flipped to the top
- moved S1 21.6 mm to (23.5, 3.17), flipped to the bottom
- moved S2 21.6 mm to (1.91, 3.17), flipped to the bottom
- moved FRAME1 20.3 mm to (22.9, -7.62), flipped to the bottom
- moved LOGO1 19.8 mm to (2.79, 2.54), flipped to the top
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Connections:
- new net N$3: J6.FEED, JP1.1
- net ANT: now also JP1.2; no longer J6.FEED
Routing:
- net 3.3V: track 111.1 -> 115.4 mm
- net N$3: track 0.00 -> 2.57 mm
- net ANT: track 11.9 -> 12.1 mm, vias 1 -> 0

Commit message: Cosmetics
Parts:
- moved U$9 26.4 mm to (-0.48, 16.9), flipped to the top
- moved U$20 25.0 mm to (0.19, 6.41), flipped to the top
- moved FD3 23.4 mm to (1.02, 13.2), flipped to the top
- moved FD4 23.4 mm to (1.02, 13.2), flipped to the bottom
- moved FD1 22.9 mm to (24.1, 44.5), flipped to the top
- moved FD2 22.9 mm to (24.1, 44.5), flipped to the bottom
- moved J1 22.9 mm to (24.1, 15.2), flipped to the top
- moved J2 22.9 mm to (1.27, 20.3), flipped to the top
- moved U$46 22.9 mm to (24.1, 10.2), flipped to the bottom
- moved J5 22.6 mm to (1.40, 15.2), flipped to the top
- moved U$45 22.6 mm to (24.0, 8.76), flipped to the bottom
- moved S1 21.6 mm to (1.91, 3.17), flipped to the top
- moved S2 21.6 mm to (23.5, 3.17), flipped to the top
- moved FRAME1 20.3 mm to (2.54, -7.62), flipped to the top
- moved LOGO1 19.8 mm to (22.6, 2.54), flipped to the bottom
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Routing:
- net 3.3V: track 115.4 -> 116.2 mm
- net RXI: track 44.7 -> 45.4 mm

Commit message: Ready for followup
Parts:
- added U$47: (no value), buzzard_labels (1):ANT_SEL0
- JP1: value JUMPER-SMT_2_NO_SILK -> Ant Sel
- U4: value RFM96W -> RFM95W; device SparkX:RFM95/96/97/98W -> SparkFun-RF:RFM95/96/97/98W
- moved U$23 3.71 mm to (21.6, 3.87), turned to 270 degrees
- moved U$22 3.69 mm to (8.26, 4.83), turned to 270 degrees
- moved R4 2.67 mm to (5.59, 5.33), turned to 0 degrees
- moved C6 2.44 mm to (3.20, 6.86)
- moved D1 1.27 mm to (5.59, 2.67)
- moved R1 1.02 mm to (7.11, 2.67)
- moved U$20 0.65 mm to (0.32, 5.78)
- moved U$36 0.53 mm to (3.40, 16.8), turned to 0 degrees
- moved D2 0.38 mm to (18.9, 2.54)
- moved R3 0.38 mm to (20.4, 2.54)
- moved S1 0.38 mm to (1.91, 2.79)
- moved S2 0.28 mm to (23.6, 2.92)
- moved R2 0.25 mm to (17.5, 2.54)
- moved J6 0.21 mm to (6.55, 16.8)
- moved U$9 0.13 mm to (-0.48, 16.8)
Routing:
- net 3.3V: track 116.2 -> 108.6 mm, vias 6 -> 7
- net 0: track 32.4 -> 33.1 mm
- net ANT: track 12.1 -> 11.4 mm
