File: Hardware/ESP32_LoRa_1_Channel_Gateway.sch (EAGLE design)
At the start: 39 parts, among them J3 USB, J4 QWIIC, J6 U.FL, Q1 MBT3904DW1T1, U1 3.3V, U2 CH340C, U3 ESP-WROOM-32NARROW, U4 RFM96W

Commit message: Made changes from REDS review pt 1
Parts:
- added JP1: JUMPER-SMT_2_NO_SILK, SparkFun-Jumpers:JUMPER-SMT_2_NO_SILK
Connections:
- new net N$3: J6.SIGNAL, JP1.1
- net ANT: now also JP1.2; no longer J6.SIGNAL
Changed lines of the file:
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@@
 <part name="C3" library="SparkFun-Capacitors" deviceset="0.1UF" device="-0603-25V-5%" value="0.1uF"/>
 <part name="LOGO5" library="SparkFun-Aesthetics" deviceset="SFE_LOGO_NAME_FLAME" device=".1_INCH" value="SFE_LOGO_NAME_FLAME.1_INCH"/>
+<part name="JP1" library="SparkFun-Jumpers" deviceset="JUMPER-SMT_2_NO" device="_SILK"/>
 </parts>
 <sheets>
@@
 <instance part="C3" gate="G$1" x="132.08" y="154.94"/>
 <instance part="LOGO5" gate="G$1" x="160.02" y="38.1"/>
+<instance part="JP1" gate="G$1" x="127" y="71.12"/>
 </instances>
 <busses>
@@
 </segment>
 <segment>
-<pinref part="J6" gate="G$1" pin="SIGNAL"/>
-<wire x1="119.38" y1="71.12" x2="121.92" y2="71.12" width="0.1524" layer="91"/>
-<label x="121.92" y="71.12" size="1.27" layer="95" xref="yes"/>
+<wire x1="132.08" y1="71.12" x2="134.62" y2="71.12" width="0.1524" layer="91"/>
+<label x="134.62" y="71.12" size="1.27" layer="95" xref="yes"/>
+<pinref part="JP1" gate="G$1" pin="2"/>
 </segment>
 <segment>
@@
 </segment>
 </net>
+<net name="N$3" class="0">
+<segment>
+<pinref part="JP1" gate="G$1" pin="1"/>
+<pinref part="J6" gate="G$1" pin="SIGNAL"/>
+<wire x1="121.92" y1="71.12" x2="119.38" y2="71.12" width="0.1524" layer="91"/>
+</segment>
+</net>

Commit message: Ready for followup
Parts:
- JP1: value JUMPER-SMT_2_NO_SILK -> Ant Sel
- U4: value RFM96W -> RFM95W; device SparkX:RFM96W -> SparkFun-RF:RFM95W
Other:
- note added: "Open this jumper if using wire antenna"
